File: hellen121vag.kicad_sch (KiCad schematic)
At the start: 111 parts, among them J1 USB_B_Mini, J10 AudioJack_THR, J2 Conn_01x01, J3 Conn_01x01, J4 Conn_01x01, J5 Conn_01x01, J6 Conn_01x01, J7 Conn_01x08, J8 Conn_01x06, M11 Module-vr-discrete-0.4, M3 mega-mcu144-0.1, M5 Module-knock-0.2, M6 Module-output-0.3, M7 Module-ign8-0.2, M8 Module-power_12and5V-0.1, M9 Module-wbo-0.5, P1 368255-2, P10 Pad, P11 Pad, P12 Pad, P13 Pad, P14 Pad, P15 Pad, P16 Pad, P17 Pad, P2 Pad, P20 Pad, P28 Pad, P3 Pad, P4 Pad, P40 Pad, P41 Pad, P43 Pad, P44 Pad, P45 Pad, P46 Pad, P48 Pad, P49 Pad, P5 Pad, P56 Pad, P6 Pad, P61 Pad, P63 Pad, P64 Pad, P66 Pad, P67 Pad, P68 Pad, P69 Pad, P7 Pad, P74 Pad, P8 Pad, P80 Pad, P9 Pad, U1 L6205PD, U3 MCP6002-xSN

Commit message: Add files via upload
Parts:
- removed D13, D14: B5819W, Diode_SMD:D_SOD-123, symbol hellen-one-common:1N4148WS
- removed J7: Conn_01x08, Connector_PinHeader_2.54mm:PinHeader_1x08_P2.54mm_Vertical, symbol Connector_Generic:Conn_01x08
- removed M11: Module-vr-discrete-0.4, hellen-one-vr-discrete-0.4:vr-discrete, symbol vr-discrete-0.4:Module-vr-discrete-0.4
- removed M3: mega-mcu144-0.1, hellen-one-mega-mcu144-0.1:mega-mcu144, symbol mega-mcu144-0.1:mega-mcu144-0.1
- removed M5: Module-knock-0.2, hellen-one-knock-0.2:knock, symbol hellen-one-knock-0.2:Module-knock-0.2
- removed M6: Module-output-0.3, hellen-one-output-0.3:output, symbol hellen-one-output-0.3:Module-output-0.3
- removed M7: Module-ign8-0.2, hellen-one-ign8-0.2:ign8, symbol hellen-one-ign8-0.2:Module-ign8-0.2
- removed M8: Module-power_12and5V-0.1, hellen-one-power_12and5V-0.1:power_12and5V, symbol power_12and5V-0.1:Module-power_12and5V-0.1
- removed M9: Module-wbo-0.5, hellen-one-wbo-0.5:wbo, symbol hellen-one-wbo-0.5:Module-wbo-0.5
- removed P10, P11, P12, P13, P14, P15, P16, P17, P20, P28, P40, P41, P43, P44, P45, P46, P48, P49, P5, P56, P6, P61, P63, P64, P66, P67, P68, P69, P7, P74, P8, P80, P9: Pad, hellen-one-common:PAD-TH, symbol hellen-one-common:Pad
- removed R23: 0, hellen-one-common:R0603, symbol hellen-one-common:Res
- added C15, C18, C6: 100n, hellen-one-common:C0603, symbol hellen-one-common:Cap
- added J11: Conn_01x06, Connector_PinHeader_2.54mm:PinHeader_1x06_P2.54mm_Vertical, symbol Connector_Generic:Conn_01x06
- added J7, J9: Conn_01x04, Connector_PinHeader_2.54mm:PinHeader_1x04_P2.54mm_Vertical, symbol Connector_Generic:Conn_01x04
- added M1, M10: Module-can-0.1, hellen-one-can-0.1:can, symbol hellen-one-can-0.1:Module-can-0.1
- added M11: Module-vr-0.1, hellen-one-vr-0.1:vr, symbol hellen-one-vr-0.1:Module-vr-0.1
- added M12: Module-dinput4-0.1, hellen-one-dinput4-0.1:dinput4, symbol hellen-one-dinput4-0.1:Module-dinput4-0.1
- added M13: Module-sd-0.1, hellen-one-sd-0.1:sd, symbol hellen-one-sd-0.1:Module-sd-0.1
- added M2: Module-power5-0.2, hellen-one-power5-0.1:power5, symbol hellen-one-power5-0.1:Module-power5-0.1
- added M3: Module-mcu-0.2, hellen-one-mcu-0.2:mcu, symbol hellen-one-mcu-0.2:Module-mcu-0.2
- added M4: Module-input-0.1, hellen-one-input-0.1:input, symbol hellen-one-input-0.1:Module-input-0.1
- added M5: Module-knock-0.1, hellen-one-knock-0.1:knock, symbol hellen-one-knock-0.1:Module-knock-0.1
- added M6: Module-output-0.2, hellen-one-output-0.2:output, symbol hellen-one-output-0.2:Module-output-0.2
- added M7: Module-ign8-0.1, hellen-one-ign8-0.1:ign8, symbol hellen-one-ign8-0.1:Module-ign8-0.1
- added M8: Module-power12-0.2, hellen-one-power12-0.2:power12, symbol hellen-one-power12-0.2:Module-power12-0.2
- added M9: Module-wbo-0.1, hellen-one-wbo-0.1:wbo, symbol hellen-one-wbo-0.1:Module-wbo-0.1
- added R14, R15: DNP, hellen-one-common:R1206, symbol hellen-one-common:Res
- added R18, R19: 4.7k, hellen-one-common:R0603, symbol hellen-one-common:Res
- added R6, R7: 2.7k, hellen-one-common:R0603, symbol hellen-one-common:Res
- added S1, S2: Button_SPST, hellen-one-common:SMD-2_2.9x3.9x1.7, symbol hellen-one-common:Button_SPST
- added U2: LPS25HB, Package_LGA:ST_HLGA-10_2.5x2.5mm_P0.6mm_LayoutBorder3x2y, symbol Sensor_Pressure:LPS25HB
- added U4: LIS2DW12TR, hellen-one-common:LGA-12_2x2mm_P0.5mm, symbol hellen-one-common:LIS2DW12TR
- added V10, V11, V12, V13, V14, V17, V20, V28, V40, V41, V43, V44, V45, V46, V48, V49, V56, V61, V63, V64, V66, V67, V68, V69, V74, V80, V9, VIN1, VIN2, VIN3, VIN4, VOUT1, VOUT2, VOUT3: Pad, hellen-one-common:PAD-TH, symbol hellen-one-common:Pad
- D10, D11, D12: value B5819W -> 1N4148WS; footprint Diode_SMD:D_SOD-123 -> hellen-one-common:SOD-323; LCSC C8598 -> C2128
- F1: LCSC (none) -> C182446; MyComment DNP -> (none)
Connections:
- net +5VP is gone; now on net +5VA: P1.53, P1.72, P1.73, P1.83, P1.98
- net +12V: now also J2.1 (Pin_1), M2.V1 (V12), M8.V1 (V12)
- net +12V_PROT: now also D10.1 (K), D11.1 (K), D12.1 (K), M6.W5 (V12P)
- net +12V_RAW: now also M6.S11 (V12_RAW), M8.E2 (V12_RAW); no longer D10.1 (K), D11.1 (K), D12.1 (K), J2.1 (Pin_1)
- net +3V3: now also C15.2, C18.2, J11.1 (Pin_1), M13.V1 (V33), M3.N16 (V33), R18.1, R19.1, S1.2, U2.1 (VDDio), U2.10 (VDD), U2.6 (~CS), U4.10 (Vdd_IO), U4.9 (Vdd)
- net +5V: now also M1.V1 (V5), M10.V1 (V5), M11.N1 (V5), M12.V1 (V5), M2.V2 (V5), M3.S1 (V5), M4.E2 (V5), M6.W14 (V5), M8.E1 (V5), M9.W1 (V5_IN)
- net +5VA: now also M3.S33 (V5A), M4.E5 (V5A), M4.J1 (PULL_V5A), M4.J10 (PULL_AUX1), M4.J17 (PULL_CAM), M4.J18 (PULL_VSS), M4.J19 (PULL_TPS), M4.J20 (PULL_O2S), M4.J21 (PULL_CRANK), M4.J5 (PULL_PPS), M4.J7 (PULL_AUX4), M4.J9 (PULL_AUX2), M4.N1 (V5A), M5.E1 (V5A), R6.2, R7.2
- net +ETB: now also M3.E14 (OUT_PWM2)
- net -ETB: now also M3.E15 (OUT_PWM3)
- net CAN+: now also M1.S2 (CANH), M10.S2 (CANH)
- net CAN-: now also M1.S1 (CANL), M10.S1 (CANL)
- net CHECK_ENGINE: now also M3.E22 (OUT_IO8), M6.W25 (LOW6_DIODE)
- net ETB_EN: now also M3.E13 (OUT_IO12)
- net FUEL_CONSUM: now also M3.E19 (OUT_PWM7), M6.W22 (PP2)
- net FUEL_PUMP_RELAY: now also M3.E8 (OUT_IO1), M6.W35 (LOW11)
- net GND: now also J1.5 (GND), C15.1, C18.1, C6.1, J11.6 (Pin_6), M1.E1 (GND), M10.E1 (GND), M11.G (GND), M12.G (GND), M12.J1 (PULL_D1), M12.J2 (PULL_D2), M12.J3 (PULL_D3), M12.J4 (PULL_D4), M13.G (GND), M13.V2 (GND), M13.V3 (GND), M2.G (GND), M3.S2 (GND), M4.E1 (GND), M5.E2 (GND), M6.G (GND), M6.S3 (GND), M7.G (GND), M8.S1 (GND), M9.E6 (LSU_H-), M9.G (GND), S2.2, U2.3 (GND), U2.5 (SA0/MISO), U2.8 (GND), U2.9 (GND), U4.6 (GND), U4.7 (RES), U4.8 (GND)
- net GNDA: now also M3.S32 (GNDA), M4.J11 (PULL_RES3), M4.J12 (PULL_MAP3), M4.J13 (PULL_MAP2), M4.J14 (PULL_MAP1), M4.J2 (PULL_GNDA), M4.J22 (PULL_KNOCK), M4.J24 (PULL_SENS3), M4.J3 (PULL_RES2), M4.J4 (PULL_O2S2), M4.J6 (PULL_RES1), M4.J8 (PULL_AUX3), M4.N2 (GNDA)
- net IDLE: now also M3.E18 (OUT_PWM6), M6.W38 (LOW3_DUAL)
- net IGN1: now also M3.W1 (OUT_IGN1), M7.V8 (IGN1)
- net IGN2: now also M3.W2 (OUT_IGN2), M7.V7 (IGN2)
- net IGN3: now also M3.W3 (OUT_IGN3), M7.V6 (IGN3)
- net IGN4: now also M3.W4 (OUT_IGN4), M7.V5 (IGN4)
- net IGN5: now also M3.W5 (OUT_IGN5), M7.V4 (IGN5)
- net IGN6: now also M3.W6 (OUT_IGN6), M7.V3 (IGN6)
- net IGN7: now also M3.W7 (OUT_IGN7), M7.V2 (IGN7)
- net IGN8: now also M3.W8 (OUT_IGN8), M7.V1 (IGN8)
- net IGN_V33: now also M3.W10 (IGN_V33), M7.V10 (V33)
- net IGN_V5: now also M3.W9 (IGN_V5), M7.V9 (VCC)
- net INJ1: now also M3.E25 (OUT_INJ1), M6.W24 (INJ1)
- net INJ2: now also M3.E26 (OUT_INJ2), M6.W23 (INJ2)
- net INJ3: now also M3.E29 (OUT_INJ3), M6.W20 (INJ3)
- net INJ4: now also M3.E30 (OUT_INJ4), M6.W19 (INJ4)
- net INJ5: now also M3.E31 (OUT_INJ5), M6.W18 (INJ5)
- net INJ6: now also M3.E32 (OUT_INJ6), M6.W17 (INJ6)
- net INJ7: now also M3.E33 (OUT_INJ7), M6.W16 (INJ7)
- net INJ8: now also M3.E34 (OUT_INJ8), M6.W15 (INJ8)
- net IN_A1: now also M4.S25 (IN_O2S2), VIN1.1 (Pin_1); no longer P2.1 (Pin_1)
- net IN_A2: now also M4.S19 (IN_MAP3), VIN2.1 (Pin_1); no longer P4.1 (Pin_1)
- net IN_A3: now also M4.S20 (IN_AUX3), VIN3.1 (Pin_1)
- net IN_A4: now also M4.S22 (IN_RES3), VIN4.1 (Pin_1); no longer P3.1 (Pin_1)
- net IN_AFR: now also M4.S9 (IN_O2S), V14.1 (Pin_1)
- net IN_CAM1: now also M4.S5 (IN_CAM)
- net IN_CAM2: now also M4.S21 (IN_AUX4)
- net IN_CLT: now also M4.S15 (IN_CLT), R6.1
- net IN_CRANK: now also M11.W2 (OUT_VR1), M4.S8 (IN_CRANK), R14.2
- net IN_CRANK+: now also M11.E2 (IN_VR1+), R14.1
- net IN_CRANK-: now also M11.E1 (IN_VR1-), R15.1
- net IN_D1: now also M12.V2 (IN_D1)
- net IN_D2: now also M12.V3 (IN_D2)
- net IN_D3: now also M12.V4 (IN_D3)
- net IN_D4: now also M12.V5 (IN_D4)
- net IN_IAT: now also M4.S16 (IN_IAT), R7.1
- net IN_KNOCK1: now also M4.S7 (IN_KNOCK), M5.E3 (OUT_KNOCK)
- net IN_KNOCK1_RAW: now also M5.W1 (IN_KNOCK)
- net IN_MAF: now also M4.S11 (IN_MAP1)
- net IN_MAP2: now also M4.S12 (IN_MAP2)
- net IN_PPS1: now also M4.S24 (IN_PPS)
- net IN_PPS2: now also M4.S18 (IN_AUX2)
- net IN_RES1: now also M4.S23 (IN_RES1)
- net IN_RES2: now also M4.S26 (IN_RES2)
- net IN_TPS1: now also M4.S10 (IN_TPS)
- net IN_TPS2: now also M4.S17 (IN_AUX1)
- net IN_VIGN: now also M8.V3 (IN_VIGN)
- net IN_VSS: now also M4.S6 (IN_VSS)
- net LSU_CALIBR_RES: now also M9.E4 (LSU_Rtrim)
- net LSU_HEAT-: now also M9.E5 (LSU_H+)
- net LSU_PUMP_I: now also M9.E3 (LSU_Ip)
- net LSU_SENSOR_U: now also M9.E1 (LSU_Un)
- net LSU_SENSOR_U/PUMP_I: now also M9.E2 (LSU_Vm)
- net MAIN_RELAY: now also M3.E6 (OUT_IO3), M6.W40 (LOW5_MAIN)
- net OUT1: now also M3.E7 (OUT_IO5), M6.W39 (LOW7_HIGH1)
- net OUT2: now also M3.E9 (OUT_IO6), M6.W37 (LOW8_HIGH2)
- net OUT3: now also M3.E28 (OUT_PWM8), M6.W21 (LOW1)
- net OUT_CHECK_ENGINE: now also M6.W3 (OUT_LOW6_DIODE)
- net OUT_FUEL_CONSUM: now also M6.S6 (OUT_PP2)
- net OUT_FUEL_PUMP_RELAY: now also M6.S10 (OUT_LOW11)
- net OUT_IDLE: now also M6.S7 (OUT_LOW3_DUAL)
- net OUT_IGN1: now also M7.S8 (OUT_IGN1)
- net OUT_IGN2: now also M7.S7 (OUT_IGN2)
- net OUT_IGN3: now also M7.S6 (OUT_IGN3)
- net OUT_IGN4: now also M7.S5 (OUT_IGN4)
- net OUT_IGN5: now also M7.S4 (OUT_IGN5)
- net OUT_IGN6: now also M7.S3 (OUT_IGN6)
- net OUT_IGN7: now also M7.S2 (OUT_IGN7)
- net OUT_IGN8: now also M7.S1 (OUT_IGN8)
- net OUT_INJ1: now also M6.S18 (OUT_INJ1)
- net OUT_INJ2: now also M6.S16 (OUT_INJ2)
- net OUT_INJ3: now also M6.S17 (OUT_INJ3)
- net OUT_INJ4: now also M6.W7 (OUT_INJ4)
- net OUT_INJ5: now also M6.W10 (OUT_INJ5)
- net OUT_INJ6: now also M6.S15 (OUT_INJ6)
- net OUT_INJ7: now also M6.W12 (OUT_INJ7)
- net OUT_INJ8: now also M6.W11 (OUT_INJ8)
- net OUT_MAIN_RELAY: now also M6.W13 (OUT_LOW5_MAIN)
- net OUT_TACH: now also M6.W6 (OUT_PP1)
- net OUT_VVT1_1: now also M6.S13 (OUT_LOW12), M6.S14 (OUT_LOW9)
- net OUT_VVT1_2: now also M6.W1 (OUT_LOW2), M6.W2 (OUT_LOW10)
- net OUT_VVT2_B1: now also M6.S5 (OUT_SOLENOID_B2)
- net OUT_VVT2_B2: now also M6.S4 (OUT_SOLENOID_B1)
- net OUT_WASTEGATE: now also M6.W4 (OUT_LOW4_DUAL)
- net RX1: now also J7.3 (Pin_3), M3.N5 (UART1_RX)
- net RX2: now also J7.1 (Pin_1), M3.N7 (UART2_RX)
- net SPI3_CS: now also J9.4 (Pin_4), M3.N8 (SPI3_CS)
- net SPI3_MISO: now also J9.2 (Pin_2), M3.N10 (SPI3_MISO)
- net SPI3_MOSI: now also J9.1 (Pin_1), M3.N11 (SPI3_MOSI)
- net SPI3_SCK: now also J9.3 (Pin_3), M3.N9 (SPI3_SCK)
- net TACH: now also M3.E27 (OUT_PWM1), M6.W28 (PP1)
- net TX1: now also J7.4 (Pin_4), M3.N4 (UART1_TX)
- net TX2: now also J7.2 (Pin_2), M3.N6 (UART2_TX)
- net USBM: now also M3.N31 (USB1M)
- net USBP: now also M3.N30 (USB1P)
- net V12_PERM: now also M8.V4 (V12_PERM)
- net VBAT: now also M3.N17 (VBAT), M8.V2 (VBAT)
- net VBUS: now also M3.N29 (VBUS)
- net VIGN: now also M3.S7 (VIGN), M8.V5 (VIGN)
- net VREF2: now also M4.S13 (VREF2), M5.W2 (VREF)
- net VVT1_1: now also M3.E10 (OUT_IO10), M6.W27 (LOW9), M6.W36 (LOW12)
- net VVT1_2: now also M3.E21 (OUT_IO7), M6.W26 (LOW10), M6.W29 (LOW2)
- net VVT2_B1: now also M3.E17 (OUT_PWM5), M6.W30 (SOLENOID_B2)
- net VVT2_B2: now also M3.E16 (OUT_PWM4), M6.W31 (SOLENOID_B1)
- net WASTEGATE: now also M3.E12 (OUT_IO2), M6.W34 (LOW4_DUAL)
- net at P1.10: now also V10.1 (Pin_1)
- net IN_KNOCK2_RAW: now reaches P1.107
- net at P1.11: now also V11.1 (Pin_1)
- net at P1.12: now also V12.1 (Pin_1)
- net at P1.13: now also V13.1 (Pin_1)
- net at P1.17: now also V17.1 (Pin_1)
- net at P1.20: now also V20.1 (Pin_1)
- net at P1.28: now also V28.1 (Pin_1)
- net at P1.40: now also V40.1 (Pin_1)
- net at P1.41: now also V41.1 (Pin_1)
- net at P1.43: now also V43.1 (Pin_1)
- net at P1.44: now also V44.1 (Pin_1)
- net at P1.45: now also V45.1 (Pin_1)
- net at P1.46: now also V46.1 (Pin_1)
- net at P1.48: now also V48.1 (Pin_1)
- net at P1.49: now also V49.1 (Pin_1)
- net at P1.56: now also V56.1 (Pin_1)
- net at P1.61: now also V61.1 (Pin_1)
- net at P1.63: now also V63.1 (Pin_1)
- net at P1.64: now also V64.1 (Pin_1)
- net at P1.66: now also V66.1 (Pin_1)
- net at P1.67: now also V67.1 (Pin_1)
- net at P1.68: now also V68.1 (Pin_1)
- net at P1.69: now also V69.1 (Pin_1)
- net at P1.74: now also V74.1 (Pin_1)
- net at P1.80: now also V80.1 (Pin_1)
- net at P1.9: now also V9.1 (Pin_1)
- net at J1.6 (Shield): no longer J1.5 (GND)
- net at J8.5 (Pin_5): now also M9.W5 (nReset)
- net at J8.4 (Pin_4): now also M9.W6 (SWDIO)
- net at J8.2 (Pin_2): now also M9.W7 (SWCLK)
- net at J8.1 (Pin_1): now also M9.W8 (V33_OUT)
- new net: M6.S12 (OUT_LOW8_PULLUP), VOUT2.1 (Pin_1)
- new net: M6.S8 (OUT_LOW1), VOUT3.1 (Pin_1)
- new net: M3.N18 (I2C_SDA), R19.2, U2.4 (SDA/MOSI)
- new net: M3.N19 (I2C_SCL), R18.2, U2.2 (SCL/SCLK)
- new net: M6.W9 (OUT_LOW7_PULLUP), VOUT1.1 (Pin_1)
- new net: M10.V2 (CAN_VIO), M9.W2 (CAN_VIO)
- new net: M10.V6 (CAN_RX), M9.W3 (CAN_RX)
- new net: M10.V5 (CAN_TX), M9.W4 (CAN_TX)
- new net A1: M3.S30 (IN_O2S2), M4.N4 (O2S2)
- new net A2: M3.S22 (IN_MAP3), M4.N12 (MAP3)
- new net A3: M3.S26 (IN_AUX3), M4.N8 (AUX3)
- new net A4: M3.S23 (IN_RES3), M4.N11 (RES3)
- new net AFR: M3.S16 (IN_O2S), M4.N18 (O2S)
- new net BOOT0: M3.N28 (BOOT0), S1.1
- new net CAM1: M3.S15 (IN_CAM), M4.N19 (CAM), P3.1 (Pin_1)
- new net CAM2: M3.S27 (IN_AUX4), M4.N7 (AUX4), P4.1 (Pin_1)
- new net CAN_RX: M1.V6 (CAN_RX), M3.N2 (CAN_RX)
- new net CAN_TX: M1.V5 (CAN_TX), M3.N3 (CAN_TX)
- new net CAN_VIO: M1.V2 (CAN_VIO), M3.N1 (CAN_VIO)
- new net CLT: M3.S18 (IN_CLT), M4.N16 (CLT)
- new net CRANK: M3.S13 (IN_CRANK), M4.N21 (CRANK), P2.1 (Pin_1)
- new net D1: M12.W4 (OUT_D1), M3.S3 (IN_D1)
- new net D2: M12.W3 (OUT_D2), M3.S4 (IN_D2)
- new net D3: M12.W2 (OUT_D3), M3.S5 (IN_D3)
- new net D4: M12.W1 (OUT_D4), M3.S6 (IN_D4)
- new net IAT: M3.S19 (IN_IAT), M4.N15 (IAT)
- new net IN_KNOCK2: M4.S3 (IN_SENS3)
- new net IO1: M3.N12 (IO1)
- new net IO2: M3.N13 (IO2)
- new net IO3: M3.N14 (IO3)
- new net IO4: M3.N15 (IO4)
- new net KNOCK1: M3.S12 (IN_KNOCK), M4.N22 (KNOCK)
- new net KNOCK2: M4.N24 (SENS3)
- new net MAF: M3.S20 (IN_MAP1), M4.N14 (MAP1)
- new net MAP2: M3.S21 (IN_MAP2), M4.N13 (MAP2)
- new net NRESET: C6.2, M3.N24 (nReset), S2.1
- new net PPS1: M3.S29 (IN_PPS), M4.N5 (PPS)
- new net PPS2: M3.S25 (IN_AUX2), M4.N9 (AUX2)
- new net RES1: M3.S28 (IN_RES1), M4.N6 (RES1)
- new net RES2: M3.S31 (IN_RES2), M4.N3 (RES2)
- new net SD_CS: J11.2 (Pin_2), M13.V4 (SD_CS), M3.N23 (SPI2_CS)
- new net SD_MISO: J11.5 (Pin_5), M13.V7 (SD_MISO), M3.N21 (SPI2_MISO)
- new net SD_MOSI: J11.3 (Pin_3), M13.V5 (SD_MOSI), M3.N22 (SPI2_MOSI)
- new net SD_SCK: J11.4 (Pin_4), M13.V6 (SD_SCK), M3.N20 (SPI2_SCK)
- new net SPI1_CS: M3.E4 (SPI1_CS1), U4.2 (~CS)
- new net SPI1_MISO: M3.E2 (SPI1_MISO), U4.3 (SA0/SDO)
- new net SPI1_MOSI: M3.E3 (SPI1_MOSI), U4.4 (SDA/SDI)
- new net SPI1_SCK: M3.E1 (SPI1_SCK), U4.1 (SCL/SPC)
- new net TPS1: M3.S17 (IN_TPS), M4.N17 (TPS)
- new net TPS2: M3.S24 (IN_AUX1), M4.N10 (AUX1)
- new net VREF1: M4.S14 (VREF1), R15.2
- new net VSS: M3.S14 (IN_VSS), M4.N20 (VSS)
- no-connect marks 70 -> 62
Other:
- note added: "Accelerometer"
- note added: "Baro"
- note removed: "#1"
- note removed: "TODO: knock 2"
- moved on the sheet: BT1, C1, C10, C11, C12, C13, C14, C16, C17, C2, C3, C4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
