File: hellen121vag.kicad_pcb (KiCad board)
At the start: 4 copper layers, 164 x 118 mm, 129 parts, among them J1 USB_B_Mini, J10 AudioJack_THR, J2 Conn_01x01, J3 Conn_01x01, J4 Conn_01x01, J5 Conn_01x01, J6 Conn_01x01, J7 Conn_01x08, J8 Conn_01x06, M1 Module-can-0.1, M10 Module-can-0.1, M11 Module-vr-discrete-0.1, M2 Module-power5-0.2, M3 Module-mcu-0.7, M4 Module-input-0.1, M5 Module-knock-0.1, M6 Module-output-0.3, M7 Module-ign8-0.2, M8 Module-power12-0.2, M9 Module-wbo-0.3, P1 368255-2, P10 Pad, P11 Pad, P12 Pad, P13 Pad, P14 Pad, P15 Pad, P16 Pad, P17 Pad, P2 Pad, P20 Pad, P28 Pad, P3 Pad, P4 Pad, P40 Pad, P41 Pad, P43 Pad, P44 Pad, P45 Pad, P46 Pad, P48 Pad, P49 Pad, P5 Pad, P56 Pad, P6 Pad, P61 Pad, P63 Pad, P64 Pad, P66 Pad, P67 Pad, P68 Pad, P69 Pad, P7 Pad, P74 Pad, P8 Pad, P80 Pad, P9 Pad, U1 L6205PD, U2 LPS25HB, U3 MCP6002-xSN, U4 TLS115_SOIC, U5 TLS115_SON

Commit message: Add files via upload
Parts:
- removed C18, C19: 1u, hellen-one-common:C0603
- removed U4: TLS115_SOIC, kicad6-libraries:PG-DSO-8-43_VIA
- removed U5: TLS115_SON, Package_SON:HVSON-8-1EP_3x3mm_P0.65mm_EP1.6x2.4mm
